File: EPS_V1_battery_pack_1.kicad_sch (KiCad schematic)
At the start: 31 parts, among them U1 MP2672AGD-0000-Z, U5 MAX17205G+

Commit message: Clean up & add labels
Other:
- note added: "CHARGER"
- note added: "FUEL GAUGE"
- moved on the sheet: C_BATT1, C_BATT2, C_BST1, C_IN1, C_REG2, C_REG3, C_SYS1, C_SYS2, C_VCC1, D_ALRT1, D_SCL1, D_SDA1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

Commit message: Add notes from Harvey meeting
Other:
- note added: "Find something in datasheet that sets pulse period/initiates a reading Likely an I2C"
- note added: "Move resistors except for R_NTC onto EPS, measure from node between R2 and RNTC"
