File: EPS_V1_battery_pack_1.kicad_sch (KiCad schematic)
At the start: 33 parts, among them U1 MP2672AGD-0000-Z, U5 MAX17205G+

Commit message: Do layout draft
Parts:
- removed D_ALRT1: 4.7, Diode_SMD:D_0603_1608Metric, symbol Device:D_Zener
- removed R_ALRT1: 1k, Resistor_SMD:R_0603_1608Metric, symbol Device:R_US
- NT2, NT3: footprint NetTie:NetTie-2_SMD_Pad2.0mm -> NetTie:NetTie-2_SMD_Pad0.5mm
Connections:
- net ALRT: now also U5.8 (ALRT1)
Other:
- moved on the sheet: D_SCL1, D_SDA1, R_SCL1, R_SDA1
