File: EPS_V1_converters.kicad_sch (KiCad schematic)
At the start: 30 parts, among them U2 TPS62132RGTR, U3 TPS62133RGTR, U6 TPS61088RHLR

Commit message: Clean up & add labels
Other:
- note added: "OUTPUT VOLTAGE REGULATORS"
- moved on the sheet: C1, C2, C3, C4, C4a1, C4b1, C5, C6, C7, C9, C_AVIN1, C_AVIN2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

Commit message: Add power switching IC
Changed lines of the file:
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@@
 	)
 	(global_label "CHG_OUT"
-		(shape passive)
+		(shape input)
 		(at 26.67 116.84 180)
 		(fields_autoplaced yes)
@@
 		)
 		(property "Intersheetrefs" "${INTERSHEET_REFS}"
-			(at 16.3294 116.84 0)
+			(at 15.2181 116.84 0)
 			(hide yes)
 			(show_name no)

Commit message: Do layout draft
Parts:
- NT1: footprint NetTie:NetTie-2_SMD_Pad2.0mm -> NetTie:NetTie-2_SMD_Pad0.5mm
Connections:
- net +12V: now reaches C4.1, C4a1.1, C4b1.1, C9.1, R1.1, U6.14 (VOUT), U6.15 (VOUT), U6.16 (VOUT)
- net +5V: now reaches C_OUT1.2, L_SW1.2, U3.14 (VOS)
- net +3V3: now reaches C_OUT2.2, L_SW2.2, U2.14 (VOS)
