File: EPS_V1_converters.kicad_sch (KiCad schematic)
At the start: 30 parts, among them U2 TPS62132RGTR, U3 TPS62133RGTR, U6 TPS61088RHLR

Commit message: Relink footprint references to consolidated libs/footprints.pretty
Parts:
- L1, L_SW1, L_SW2: footprint IFSC1515AHER2R2M01:IND_IFSC_1515AH_VIS -> footprints:IND_IFSC_1515AH_VIS
- U2: footprint TPS62132RGTR:RGT16_1P7X1P7 -> footprints:RGT16_1P7X1P7
- U3: footprint TPS62133RGTR:RGT0016C -> footprints:RGT0016C
- U6: footprint TPS61088RHLR:RHL0020A -> footprints:RHL0020A
Changed lines of the file:
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@@
 			)
 		)
-		(property "Footprint" "TPS62133RGTR:RGT0016C"
+		(property "Footprint" "footprints:RGT0016C"
 			(at 99.06 124.46 0)
 			(hide yes)
@@
 			)
 		)
-		(property "Footprint" "IFSC1515AHER2R2M01:IND_IFSC_1515AH_VIS"
+		(property "Footprint" "footprints:IND_IFSC_1515AH_VIS"
 			(at 133.35 134.62 0)
 			(hide yes)
@@
 			)
 		)
-		(property "Footprint" "TPS62132RGTR:RGT16_1P7X1P7"
+		(property "Footprint" "footprints:RGT16_1P7X1P7"
 			(at 129.54 173.99 0)
 			(hide yes)
@@
 			)
 		)
-		(property "Footprint" "TPS61088RHLR:RHL0020A"
+		(property "Footprint" "footprints:RHL0020A"
 			(at 87.63 67.31 0)
 			(hide yes)
@@
 			)
 		)
-		(property "Footprint" "IFSC1515AHER2R2M01:IND_IFSC_1515AH_VIS"
+		(property "Footprint" "footprints:IND_IFSC_1515AH_VIS"
 			(at 133.35 173.99 0)
 			(hide yes)
@@
 			)
 		)
-		(property "Footprint" "IFSC1515AHER2R2M01:IND_IFSC_1515AH_VIS"
+		(property "Footprint" "footprints:IND_IFSC_1515AH_VIS"
 			(at 87.63 29.21 0)
 			(hide yes)
