File: EPS_V1_battery_pack_3.kicad_sch (KiCad schematic)
At the start: 31 parts, among them U10 MP2672AGD-0000-Z, U11 MAX17205G+

Commit message: Relink footprint references to consolidated libs/footprints.pretty
Parts:
- L_3: footprint AMELA2012S_1R5MT:IND_AMELA2012S-1R5MT -> footprints:IND_AMELA2012S-1R5MT
- U10: footprint MP2672AGD_0000_Z:QFN-18_MP2672A_MNP -> footprints:QFN-18_MP2672A_MNP
- U11: footprint MAX17205G:21-0137_T1433&plus_2C_MXM -> footprints:21-0137_T1433&plus_2C_MXM
Changed lines of the file:
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@@
 			)
 		)
-		(property "Footprint" "MP2672AGD_0000_Z:QFN-18_MP2672A_MNP"
+		(property "Footprint" "footprints:QFN-18_MP2672A_MNP"
 			(at 63.5 78.74 0)
 			(hide yes)
@@
 			)
 		)
-		(property "Footprint" "MAX17205G:21-0137_T1433&plus_2C_MXM"
+		(property "Footprint" "footprints:21-0137_T1433&plus_2C_MXM"
 			(at 184.15 74.93 0)
 			(hide yes)
@@
 			)
 		)
-		(property "Footprint" "AMELA2012S_1R5MT:IND_AMELA2012S-1R5MT"
+		(property "Footprint" "footprints:IND_AMELA2012S-1R5MT"
 			(at 58.42 72.39 0)
 			(hide yes)
