File: EPS_V1_battery_pack_4.kicad_sch (KiCad schematic)
At the start: 31 parts, among them U12 MP2672AGD-0000-Z, U13 MAX17205G+

Commit message: Relink footprint references to consolidated libs/footprints.pretty
Parts:
- L_4: footprint AMELA2012S_1R5MT:IND_AMELA2012S-1R5MT -> footprints:IND_AMELA2012S-1R5MT
- U12: footprint MP2672AGD_0000_Z:QFN-18_MP2672A_MNP -> footprints:QFN-18_MP2672A_MNP
- U13: footprint MAX17205G:21-0137_T1433&plus_2C_MXM -> footprints:21-0137_T1433&plus_2C_MXM
Changed lines of the file:
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@@
 			)
 		)
-		(property "Footprint" "AMELA2012S_1R5MT:IND_AMELA2012S-1R5MT"
+		(property "Footprint" "footprints:IND_AMELA2012S-1R5MT"
 			(at 58.42 73.66 0)
 			(hide yes)
@@
 			)
 		)
-		(property "Footprint" "MAX17205G:21-0137_T1433&plus_2C_MXM"
+		(property "Footprint" "footprints:21-0137_T1433&plus_2C_MXM"
 			(at 184.15 76.2 0)
 			(hide yes)
@@
 			)
 		)
-		(property "Footprint" "MP2672AGD_0000_Z:QFN-18_MP2672A_MNP"
+		(property "Footprint" "footprints:QFN-18_MP2672A_MNP"
 			(at 63.5 80.01 0)
 			(hide yes)
