File: EPS_V1_charging_inputs.kicad_sch (KiCad schematic)
At the start: 27 parts, among them U4 MP28167GQ-Z, U7 TPS2121RUXR

Commit message: Relink footprint references to consolidated libs/footprints.pretty
Parts:
- L2: footprint ASPI_7318_4R7M_T:IND_ASPI-7318-4R7M-T -> footprints:IND_ASPI-7318-4R7M-T
- U4: footprint MP28167GQ-Z:QFN-16_MP28167GQ_MNP -> footprints:QFN-16_MP28167GQ_MNP
- U7: footprint TPS2121RUXR:RUX0012A -> footprints:RUX0012A
Changed lines of the file:
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@@
 			)
 		)
-		(property "Footprint" "ASPI_7318_4R7M_T:IND_ASPI-7318-4R7M-T"
+		(property "Footprint" "footprints:IND_ASPI-7318-4R7M-T"
 			(at 170.18 123.19 0)
 			(hide yes)
@@
 			)
 		)
-		(property "Footprint" "TPS2121RUXR:RUX0012A"
+		(property "Footprint" "footprints:RUX0012A"
 			(at 133.35 49.53 0)
 			(hide yes)
@@
 			)
 		)
-		(property "Footprint" "MP28167GQ-Z:QFN-16_MP28167GQ_MNP"
+		(property "Footprint" "footprints:QFN-16_MP28167GQ_MNP"
 			(at 118.11 120.65 0)
 			(hide yes)
