File: schematics/EPS_V1_battery_pack_1.kicad_sch (KiCad schematic)
At the start: 31 parts, among them U1 MP2672AGD-0000-Z, U5 MAX17205G+

Commit message: Add chargers to I2C, chg_in for ADC
Parts:
- removed D_SCL1, D_SDA1: 4.7, Diode_SMD:D_0603_1608Metric, symbol Device:D_Zener
- removed R_SCL1, R_SDA1: 150R, Resistor_SMD:R_0603_1608Metric, symbol Device:R_US
Connections:
- net GND: no longer U1.14 (SCL), U1.15 (SDA)
- net I2C1_SCL: now also U1.14 (SCL), U5.11 (OD/SCL)
- net I2C1_SDA: now also U1.15 (SDA), U5.12 (DQ/SDA)

Commit message: Fix standalone to host control mode
Parts:
- removed R_VBATT1: 33k, Resistor_SMD:R_0603_1608Metric, symbol Device:R_US
Connections:
- net at U1.17 (CV): now also C_VCC1.2, R_ACOK1.2, R_STAT1.1, R_T1.1, U1.4 (VCC)
Changed lines of the file:
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@@
 	)
 	(junction
+		(at 105.41 63.5)
+		(diameter 0)
+		(color 0 0 0 0)
+	)
+	(junction
 		(at 181.61 82.55)
 		(diameter 0)
@@
 	(wire
 		(pts
-			(xy 116.84 81.28) (xy 116.84 85.09)
-		)
-		(stroke
-			(width 0)
-			(type default)
-		)
-	)
-	(wire
-		(pts
 			(xy 105.41 104.14) (xy 105.41 105.41)
 		)
@@
 	(wire
 		(pts
+			(xy 105.41 63.5) (xy 105.41 81.28)
+		)
+		(stroke
+			(width 0)
+			(type default)
+		)
+	)
+	(wire
+		(pts
 			(xy 229.87 87.63) (xy 229.87 90.17)
 		)
@@
 	(wire
 		(pts
+			(xy 104.14 81.28) (xy 105.41 81.28)
+		)
+		(stroke
+			(width 0)
+			(type default)
+		)
+	)
+	(wire
+		(pts
 			(xy 118.11 104.14) (xy 120.65 104.14)
 		)
@@
 	(wire
 		(pts
-			(xy 48.26 63.5) (xy 48.26 86.36)
+			(xy 105.41 63.5) (xy 48.26 63.5)
 		)
 		(stroke
@@
 	(wire
 		(pts
-			(xy 114.3 63.5) (xy 48.26 63.5)
+			(xy 48.26 63.5) (xy 48.26 86.36)
 		)
 		(stroke
@@
 	(wire
 		(pts
-			(xy 160.02 77.47) (xy 184.15 77.47)
+			(xy 114.3 63.5) (xy 105.41 63.5)
 		)
 		(stroke
@@
 	(wire
 		(pts
-			(xy 105.41 96.52) (xy 105.41 104.14)
+			(xy 160.02 77.47) (xy 184.15 77.47)
 		)
 		(stroke
@@
 	(wire
 		(pts
-			(xy 104.14 81.28) (xy 116.84 81.28)
+			(xy 105.41 96.52) (xy 105.41 104.14)
 		)
 		(stroke
@@
 	)
 	(symbol
-		(lib_id "Device:R_US")
-		(at 116.84 88.9 0)
-		(unit 1)
-		(body_style 1)
-		(exclude_from_sim no)
-		(in_bom yes)
-		(on_board yes)
-		(in_pos_files yes)
-		(dnp no)
-		(property "Reference" "R_VBATT1"
-			(at 118.872 87.63 0)
-			(show_name no)
-			(do_not_autoplace no)
-			(effects
-				(font
-					(size 1.27 1.27)
-				)
-				(justify left)
-			)
-		)
-		(property "Value" "33k"
-			(at 118.872 90.17 0)
-			(show_name no)
-			(do_not_autoplace no)
-			(effects
-				(font
-					(size 1.27 1.27)
-				)
-				(justify left)
-			)
-		)
-		(property "Footprint" "Resistor_SMD:R_0603_1608Metric"
-			(at 117.856 89.154 90)
-			(hide yes)
-			(show_name no)
-			(do_not_autoplace no)
-			(effects
-				(font
-					(size 1.27 1.27)
-				)
-			)
-		)
-		(property "Datasheet" ""
-			(at 116.84 88.9 0)
-			(hide yes)
-			(show_name no)
-			(do_not_autoplace no)
-			(effects
-				(font
-					(size 1.27 1.27)
-				)
-			)
-		)
-		(property "Description" "Resistor, US symbol"
-			(at 116.84 88.9 0)
-			(hide yes)
-			(show_name no)
-			(do_not_autoplace no)
-			(effects
-				(font
-					(size 1.27 1.27)
-				)
-			)
-		)
-		(pin "2"
-		)
-		(pin "1"
-		)
-		(instances
-			(project "EPS_V1"
-				(path "/85157432-5d03-48fa-ab40-27ed3d133f47/d6a7ca1d-fe68-467f-8233-74a5cf811189"
-					(reference "R_VBATT1")
-					(unit 1)
-				)
-			)
-		)
-	)
-	(symbol
 		(lib_id "power:GND")
 		(at 179.07 118.11 0)
@@
 					(unit 1)
 				)
-			)
-		)
-	)
-	(symbol
-		(lib_id "sym_lib:GNDA1")
-		(at 116.84 92.71 0)
-		(unit 1)
-		(body_style 1)
-		(exclude_from_sim no)
-		(in_bom no)
-		(on_board no)
-		(in_pos_files yes)
-		(dnp no)
-		(property "Reference" "#PWR04"
-			(at 116.84 92.71 0)
-			(hide yes)
-			(show_name no)
-			(do_not_autoplace no)
-			(effects
-				(font
-					(size 1.27 1.27)
-				)
-			)
-		)
-		(property "Value" "GNDA1"
-			(at 116.84 97.028 0)
-			(show_name no)
-			(do_not_autoplace no)
-			(effects
-				(font
-					(size 1.27 1.27)
-				)
-			)
-		)
-		(property "Footprint" ""
-			(at 116.84 92.71 0)
-			(hide yes)
-			(show_name no)
-			(do_not_autoplace no)
-			(effects
-				(font
-					(size 1.27 1.27)
-				)
-			)
-		)
-		(property "Datasheet" ""
-			(at 116.84 92.71 0)
-			(hide yes)
-			(show_name no)
-			(do_not_autoplace no)
-			(effects
-				(font
-					(size 1.27 1.27)
-				)
-			)
-		)
-		(property "Description" ""
-			(at 116.84 92.71 0)
-			(hide yes)
-			(show_name no)
-			(do_not_autoplace no)
-			(effects
-				(font
-					(size 1.27 1.27)
-				)
-			)
-		)
-		(pin "1"
-		)
-		(instances
-			(project "EPS_V1"
-				(path "/85157432-5d03-48fa-ab40-27ed3d133f47/d6a7ca1d-fe68-467f-8233-74a5cf811189"
-					(reference "#PWR04")
-					(unit 1)
-				)
